File: driver_bldc.kicad_pcb (KiCad board)
At the start: 2 copper layers, 6 parts, among them J1 Conn_01x03, Q1 BTN8982TA, Q2 BTN8982TA, Q3 BTN8982TA, U1 STM32G431CBT6, U2 SN65HVD234

Commit message: dodat buck
Parts:
- added J3: BATT, Connector_AMASS:AMASS_XT30PW-M_1x02_P2.50mm_Horizontal, F.Cu at (50.5, 43.5)
- added U3: AP63203WU, Package_TO_SOT_SMD:TSOT-23-6_HandSoldering, F.Cu at (43.8, 48.6)
- J1: value Conn_01x03 -> CAN
Connections:
- net CAN_RX renamed CAN_RX+
- net CAN_TX renamed CAN_TX-
- net Net-(Q1-Pad4) renamed A
- net Net-(Q2-Pad4) renamed B
- net Net-(Q3-Pad4) renamed C
